Commit message: Sync direct camera mount and MU ROS CAD assembly

File: ros2_sim_ws/src/fusion_model_ros2_beta/urdf/ur10_official.urdf (robot description, URDF)
Before this commit: robot ur10, 20 links, 19 joints
Links:
- removed link ati_sensor_link
- removed link mecheye_camera_link
- removed link robotiq_gripper_link
- added link cad_connector_link; collision mesh filename=package://fusion_model_ros2_beta/meshes/end_effector/end_ef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 scale=0.001 0.001 0.001; visual mesh filename=package://fusion_model_ros2_beta/meshes/end_effector/end_ef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 scale=0.001 0.001 0.001
- added link cad_force_sensor_link; collision mesh filename=package://fusion_model_ros2_beta/meshes/end_effector/end_ef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 scale=0.001 0.001 0.001; visual mesh filename=package://fusion_model_ros2_beta/meshes/end_effector/end_ef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 scale=0.001 0.001 0.001
- added link cad_mecheye_camera_link; collision mesh filename=package://fusion_model_ros2_beta/meshes/end_effector/end_ef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 scale=0.001 0.001 0.001; visual mesh filename=package://fusion_model_ros2_beta/meshes/end_effector/end_ef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 scale=0.001 0.001 0.001
- added link cad_robotiq_2f85_link; collision mesh filename=package://fusion_model_ros2_beta/meshes/end_effector/end_ef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 scale=0.001 0.001 0.001; visual mesh filename=package://fusion_model_ros2_beta/meshes/end_effector/end_ef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 scale=0.001 0.001 0.001
- added link mecheye_camera_optical_frame_legacy_20260921
Joints:
- removed joint ati_sensor-robotiq_gripper
- removed joint gripper-brush
- removed joint tool0-ati_sensor
- removed joint tool0-mecheye_camera
- added joint tool0-brush: type fixed, parent tool0, child brush_link, origin xyz=0 0 0.220 rpy=0 0 0
- added joint tool0-cad_connector: type fixed, parent tool0, child cad_connector_link, origin xyz=-0.080221162 0.327612370 0.238737610 rpy=-1.570796327 0 -1.570796327
- added joint tool0-cad_force_sensor: type fixed, parent tool0, child cad_force_sensor_link, origin xyz=-0.080221162 0.327612370 0.238737610 rpy=-1.570796327 0 -1.570796327
- added joint tool0-cad_mecheye_camera: type fixed, parent tool0, child cad_mecheye_camera_link, origin xyz=-0.080221162 0.327612370 0.238737610 rpy=-1.570796327 0 -1.570796327
- added joint tool0-cad_robotiq_2f85: type fixed, parent tool0, child cad_robotiq_2f85_link, origin xyz=-0.080221162 0.327612370 0.238737610 rpy=-1.570796327 0 -1.570796327
- added joint tool0-mecheye_camera_optical_legacy_20260921: type fixed, parent tool0, child mecheye_camera_optical_frame_legacy_20260921, origin xyz=0.0484942352 0.2520224071 0.1993161073 rpy=-1.1547020625 -0.0002532205 -3.1353642945
